Commit message: Panic save

File: ros_visualization/src/iiwa14/urdf/iiwa14_with_wall.urdf (robot description, URDF)
Before this commit: robot iiwa14, 12 links, 11 joints
Links:
- link wall_link: geometry visual box size=1 0.02 1.4
Joints:
- joint world_wall_joint: origin xyz=5 0.4 0 rpy=0 0 0.523 -> xyz=5 0.42 0 rpy=0 0 0
